File: hd44780_driver.sch (KiCad schematic (older format))
At the start: 23 parts, among them J2 BL, J3 Conn_01x08, Q1 2N7002, U1 PCA9555APW

Commit message: add a input and move VE from the expander to the connector
Parts:
- added R15: 10k, Resistor_SMD:R_0805_2012Metric_Pad1.15x1.40mm_HandSolder, symbol hd44780_driver-rescue:R-Device
- J3: value Conn_01x08 -> Conn_01x10; footprint Connector_PinHeader_2.54mm:PinHeader_1x08_P2.54mm_Vertical -> Connector_PinHeader_2.54mm:PinHeader_1x10_P2.54mm_Vertical; symbol Connector_Generic:Conn_01x08 -> Connector_Generic:Conn_01x10
- renumbered R15 to R16
Connections:
- net BUT0: now also J3.9 (Pin_9), U1.17 (P1_4); no longer J3.7 (Pin_7), U1.18 (P1_5)
- net BUT1: now also J3.8 (Pin_8), U1.18 (P1_5); no longer J3.6 (Pin_6), U1.19 (P1_6)
- net BUT2: now also J3.7 (Pin_7), U1.19 (P1_6); no longer J3.5 (Pin_5), U1.20 (P1_7)
- net VCC: now also J3.10 (Pin_10), R15.2; no longer J3.8 (Pin_8)
- net VE: now also J3.5 (Pin_5); no longer U1.17 (P1_4)
- new net BUT3: J3.6 (Pin_6), R15.1, U1.20 (P1_7)
Other:
- moved on the sheet: R12, R13, R14
Changed lines of the file:
@@
 L hd44780_driver-rescue:R-Device R12
 U 1 1 5F566099
-P 6150 2950
-F 0 "R12" V 6050 2950 50  0000 C CNN
-F 1 "10k" V 6150 2950 50  0000 C CNN
-F 2 "Resistor_SMD:R_0805_2012Metric_Pad1.15x1.40mm_HandSolder" V 6080 2950 50  0001 C CNN
-F 3 "~" H 6150 2950 50  0001 C CNN
-	1    6150 2950
+P 5950 2850
+F 0 "R12" V 5850 2850 50  0000 C CNN
+F 1 "10k" V 5950 2850 50  0000 C CNN
+F 2 "Resistor_SMD:R_0805_2012Metric_Pad1.15x1.40mm_HandSolder" V 5880 2850 50  0001 C CNN
+F 3 "~" H 5950 2850 50  0001 C CNN
+	1    5950 2850
 	-1   0    0    1
 $EndComp
@@
 Text Label 7200 3250 0    50   ~ 0
 VE
-Text Label 5500 3150 2    50   ~ 0
-VE
 $Comp
 L hd44780_driver-rescue:Logo_Open_Hardware_Small-Graphic #LOGO1
@@
 Wire Wire Line
 	5500 3050 5250 3050
-Wire Wire Line
-	5500 3150 5250 3150
 Text Label 5500 1850 2    50   ~ 0
 D0
@@
 D0
 Wire Wire Line
-	1150 2150 1450 2150
-Wire Wire Line
-	1450 1950 1150 1950
-Wire Wire Line
-	1350 1550 1150 1550
-Wire Wire Line
-	1350 1200 1350 1550
+	1150 2250 1450 2250
+Wire Wire Line
+	1450 2050 1150 2050
+Wire Wire Line
+	1350 1450 1150 1450
+Wire Wire Line
+	1350 1100 1350 1450
 $Comp
 L hd44780_driver-rescue:VCC-power #PWR05
 U 1 1 5F02A73B
-P 1350 1200
-F 0 "#PWR05" H 1350 1050 50  0001 C CNN
-F 1 "VCC" H 1367 1373 50  0000 C CNN
-F 2 "" H 1350 1200 50  0001 C CNN
-F 3 "" H 1350 1200 50  0001 C CNN
-	1    1350 1200
-	1    0    0    -1
-$EndComp
-Wire Wire Line
-	1350 2250 1150 2250
-Wire Wire Line
-	1350 2500 1350 2250
+P 1350 1100
+F 0 "#PWR05" H 1350 950 50  0001 C CNN
+F 1 "VCC" H 1367 1273 50  0000 C CNN
+F 2 "" H 1350 1100 50  0001 C CNN
+F 3 "" H 1350 1100 50  0001 C CNN
+	1    1350 1100
+	1    0    0    -1
+$EndComp
+Wire Wire Line
+	1350 2350 1150 2350
+Wire Wire Line
+	1350 2600 1350 2350
 $Comp
 L hd44780_driver-rescue:GND-power #PWR06
 U 1 1 5F02A733
-P 1350 2500
-F 0 "#PWR06" H 1350 2250 50  0001 C CNN
-F 1 "GND" H 1355 2327 50  0000 C CNN
-F 2 "" H 1350 2500 50  0001 C CNN
-F 3 "" H 1350 2500 50  0001 C CNN
-	1    1350 2500
-	1    0    0    -1
-$EndComp
-$Comp
-L Connector_Generic:Conn_01x08 J3
+P 1350 2600
+F 0 "#PWR06" H 1350 2350 50  0001 C CNN
+F 1 "GND" H 1355 2427 50  0000 C CNN
+F 2 "" H 1350 2600 50  0001 C CNN
+F 3 "" H 1350 2600 50  0001 C CNN
+	1    1350 2600
+	1    0    0    -1
+$EndComp
+$Comp
+L Connector_Generic:Conn_01x10 J3
 U 1 1 5F02A72C
 P 950 1950
 F 0 "J3" H 950 2350 50  0000 C CNN
-F 1 "Conn_01x08" V 1050 1950 50  0000 C CNN
-F 2 "Connector_PinHeader_2.54mm:PinHeader_1x08_P2.54mm_Vertical" H 950 1950 50  0001 C CNN
+F 1 "Conn_01x10" V 1050 1950 50  0000 C CNN
+F 2 "Connector_PinHeader_2.54mm:PinHeader_1x10_P2.54mm_Vertical" H 950 1950 50  0001 C CNN
 F 3 "~" H 950 1950 50  0001 C CNN
 	1    950  1950
@@
 $EndComp
 $Comp
-L hd44780_driver-rescue:R-Device R15
+L hd44780_driver-rescue:R-Device R16
 U 1 1 61615E80
 P 8650 5100
-F 0 "R15" V 8750 5100 50  0000 C CNN
+F 0 "R16" V 8750 5100 50  0000 C CNN
 F 1 "330" V 8650 5100 50  0000 C CNN
 F 2 "Resistor_SMD:R_0805_2012Metric_Pad1.15x1.40mm_HandSolder" V 8580 5100 50  0001 C CNN
@@
 L hd44780_driver-rescue:R-Device R14
 U 1 1 61615E87
-P 6550 2950
-F 0 "R14" V 6650 2950 50  0000 C CNN
-F 1 "10k" V 6550 2950 50  0000 C CNN
-F 2 "Resistor_SMD:R_0805_2012Metric_Pad1.15x1.40mm_HandSolder" V 6480 2950 50  0001 C CNN
-F 3 "~" H 6550 2950 50  0001 C CNN
-	1    6550 2950
+P 6350 2850
+F 0 "R14" V 6450 2850 50  0000 C CNN
+F 1 "10k" V 6350 2850 50  0000 C CNN
+F 2 "Resistor_SMD:R_0805_2012Metric_Pad1.15x1.40mm_HandSolder" V 6280 2850 50  0001 C CNN
+F 3 "~" H 6350 2850 50  0001 C CNN
+	1    6350 2850
 	1    0    0    1
 $EndComp
@@
 L hd44780_driver-rescue:R-Device R13
 U 1 1 61615E8E
-P 6350 2950
-F 0 "R13" V 6450 2950 50  0000 C CNN
-F 1 "10k" V 6350 2950 50  0000 C CNN
-F 2 "Resistor_SMD:R_0805_2012Metric_Pad1.15x1.40mm_HandSolder" V 6280 2950 50  0001 C CNN
-F 3 "~" H 6350 2950 50  0001 C CNN
-	1    6350 2950
-	1    0    0    1
-$EndComp
-Wire Wire Line
-	6150 2800 6150 2700
-Wire Wire Line
-	6150 2700 6350 2700
-Wire Wire Line
-	6550 2700 6550 2800
-Wire Wire Line
-	6350 2800 6350 2700
-Connection ~ 6350 2700
-Wire Wire Line
-	6350 2700 6550 2700
+P 6150 2850
+F 0 "R13" V 6250 2850 50  0000 C CNN
+F 1 "10k" V 6150 2850 50  0000 C CNN
+F 2 "Resistor_SMD:R_0805_2012Metric_Pad1.15x1.40mm_HandSolder" V 6080 2850 50  0001 C CNN
+F 3 "~" H 6150 2850 50  0001 C CNN
+	1    6150 2850
+	1    0    0    1
+$EndComp
+Wire Wire Line
+	6150 2700 6150 2600
+Wire Wire Line
+	6150 2600 6350 2600
+Wire Wire Line
+	6550 2600 6550 2700
+Wire Wire Line
+	6350 2700 6350 2600
+Connection ~ 6350 2600
+Wire Wire Line
+	6350 2600 6550 2600
 $Comp
 L hd44780_driver-rescue:VCC-power #PWR08
 U 1 1 61615E9D
-P 6350 2300
-F 0 "#PWR08" H 6350 2150 50  0001 C CNN
-F 1 "VCC" H 6367 2473 50  0000 C CNN
-F 2 "" H 6350 2300 50  0001 C CNN
-F 3 "" H 6350 2300 50  0001 C CNN
-	1    6350 2300
-	1    0    0    -1
-$EndComp
-Wire Wire Line
-	6350 2300 6350 2700
-Wire Wire Line
-	6150 3250 6150 3100
+P 6350 2200
+F 0 "#PWR08" H 6350 2050 50  0001 C CNN
+F 1 "VCC" H 6367 2373 50  0000 C CNN
+F 2 "" H 6350 2200 50  0001 C CNN
+F 3 "" H 6350 2200 50  0001 C CNN
+	1    6350 2200
+	1    0    0    -1
+$EndComp
+Wire Wire Line
+	6350 2200 6350 2600
 Wire Wire Line
 	5250 3250 6150 3250
 Wire Wire Line
-	6350 3100 6350 3350
-Wire Wire Line
 	5250 3350 6350 3350
 Wire Wire Line
-	6550 3450 6550 3100
-Wire Wire Line
 	5250 3450 6550 3450
+Text Label 5500 3150 2    50   ~ 0
+BUT0
 Text Label 5500 3250 2    50   ~ 0
-BUT0
+BUT1
 Text Label 5500 3350 2    50   ~ 0
-BUT1
-Text Label 5500 3450 2    50   ~ 0
 BUT2
 Wire Wire Line
@@
 INT
 Wire Wire Line
-	1150 2050 1450 2050
+	1150 2150 1450 2150
+Text Label 1450 2150 2    50   ~ 0
+SCL
+Text Label 1450 2250 2    50   ~ 0
+SDA
 Text Label 1450 2050 2    50   ~ 0
-SCL
-Text Label 1450 2150 2    50   ~ 0
-SDA
-Text Label 1450 1950 2    50   ~ 0
 INT
 Wire Wire Line
+	1150 1550 1450 1550
+Text Label 1450 1550 2    50   ~ 0
+BUT0
+Text Label 1450 1650 2    50   ~ 0
+BUT1
+Text Label 1450 1750 2    50   ~ 0
+BUT2
+Wire Wire Line
 	1150 1650 1450 1650
-Text Label 1450 1650 2    50   ~ 0
-BUT0
-Text Label 1450 1750 2    50   ~ 0
-BUT1
-Text Label 1450 1850 2    50   ~ 0
-BUT2
 Wire Wire Line
 	1150 1750 1450 1750
-Wire Wire Line
-	1150 1850 1450 1850
 $Comp
 L power:PWR_FLAG #FLG0101
@@
 Wire Wire Line
 	1100 7050 1100 6850
+$Comp
+L hd44780_driver-rescue:R-Device R15
+U 1 1 61A26DCB
+P 6550 2850
+F 0 "R15" V 6450 2850 50  0000 C CNN
+F 1 "10k" V 6550 2850 50  0000 C CNN
+F 2 "Resistor_SMD:R_0805_2012Metric_Pad1.15x1.40mm_HandSolder" V 6480 2850 50  0001 C CNN
+F 3 "~" H 6550 2850 50  0001 C CNN
+	1    6550 2850
+	-1   0    0    1
+$EndComp
+Wire Wire Line
+	5950 2700 5950 2600
+Wire Wire Line
+	5950 2600 6150 2600
+Connection ~ 6150 2600
+Wire Wire Line
+	5250 3150 5950 3150
+Wire Wire Line
+	5950 3000 5950 3150
+Wire Wire Line
+	6150 3000 6150 3250
+Wire Wire Line
+	6350 3000 6350 3350
+Wire Wire Line
+	6550 3000 6550 3450
+Text Label 5500 3450 2    50   ~ 0
+BUT3
+Text Label 1450 1850 2    50   ~ 0
+BUT3
+Wire Wire Line
+	1150 1850 1450 1850
+Wire Wire Line
+	1150 1950 1450 1950
+Text Label 1450 1950 2    50   ~ 0
+VE
 $EndSCHEMATC

Commit message: Change the footprint
Parts:
- U1: footprint Package_SO:TSSOP-24_4.4x7.8mm_P0.65mm -> Package_SO:SSOP-24_5.3x8.2mm_P0.65mm
Changed lines of the file:
@@
 F 0 "U1" H 4750 3740 60  0000 C CNN
 F 1 "PCA9555APW" H 4750 3634 60  0000 C CNN
-F 2 "Package_SO:TSSOP-24_4.4x7.8mm_P0.65mm" H 4250 3250 60  0001 C CNN
+F 2 "Package_SO:SSOP-24_5.3x8.2mm_P0.65mm" H 4250 3250 60  0001 C CNN
 F 3 "http://www.nxp.com/documents/data_sheet/PCA9555A.pdf" H 4750 3634 60  0001 C CNN
 	1    4750 2650
